Commit message: add kinect to main youbot urdf file

File: raw_common/raw_robot_description/urdf/tower/cam3d_tower.urdf.xacro (robot description, xacro)
@@ -4,5 +4,4 @@
        xmlns:interface="http://playerstage.sourceforge.net/gazebo/xmlschema/#interface"
        xmlns:xacro="http://ros.org/wiki/xacro">
-  <include filename="$(find raw_robot_description)/urdf/sensors/kinect.urdf.xacro" />
   <property name="height" value="0.515" />
   <property name="width" value="0.03" />
@@ -35,7 +34,3 @@
     </joint>
   </xacro:macro>
-  <!-- 3D camera on tower -->
-  <xacro:kinect name="openni" parent="tower_link">
-    <origin xyz="0.05 0 ${height}" rpy="0 0.61 0" />
-  </xacro:kinect>
 </root>

File: raw_robots/raw_hardware_config/youbot-hbrs2/urdf/youbot-hbrs2.urdf.xacro (robot description, xacro)
@@ -42,5 +42,5 @@
   <include filename="$(find raw_robot_description)/urdf/materials.urdf.xacro" />
   <include filename="$(find raw_robot_description)/urdf/tower/cam3d_tower.urdf.xacro" />
-  <!--include filename="$(find youbot_description)/urdf/sensors/asus_xtion.urdf.xacro" />-->
+  <include filename="$(find raw_robot_description)/urdf/sensors/kinect.urdf.xacro" />
   <!-- base laser rear -->
   <xacro:hokuyo_urg04_laser name="base_laser_rear" parent="base" ros_topic="scan_rear" update_rate="10" min_angle="-1.57" max_angle="1.57" >
@@ -51,8 +51,8 @@
     <origin xyz="-0.015 0 0.025" rpy="0 0 0" />
   </xacro:cam3d_tower>
-  <!-- ASUS Xtion on arm joint 4
-  <xacro:asus_xtion name="asus_xtion" parent="arm_link_4" ros_topic="/camera/rgb/points" tilt="0.0">
-    <origin xyz="0.03 0 0.055" rpy="0 -${M_PI/2} ${M_PI}" />
-  </xacro:asus_xtion>
+  <!-- 3D camera on tower -->
+  <xacro:kinect name="openni" parent="plate_link">
+    <origin xyz="-0.010 0.008 0.422" rpy="-0.048 0.419 0.031" />
+  </xacro:kinect>
   -->
 </robot>

Commit message: adjust tower/kinect pos

File: raw_common/raw_robot_description/urdf/tower/cam3d_tower.urdf.xacro (robot description, xacro)
@@ -4,5 +4,5 @@
        xmlns:interface="http://playerstage.sourceforge.net/gazebo/xmlschema/#interface"
        xmlns:xacro="http://ros.org/wiki/xacro">
-  <property name="height" value="0.515" />
+  <property name="height" value="0.49" />
   <property name="width" value="0.03" />
   <property name="depth" value="0.03" />

File: raw_robots/raw_hardware_config/youbot-hbrs2/urdf/youbot-hbrs2.urdf.xacro (robot description, xacro)
@@ -49,9 +49,9 @@
   <!-- tower with 3D camera -->
   <xacro:cam3d_tower name="tower" parent="plate_link">
-    <origin xyz="-0.015 0 0.025" rpy="0 0 0" />
+    <origin xyz="-0.0659 0.0 0.025" rpy="0 0 0" />
   </xacro:cam3d_tower>
   <!-- 3D camera on tower -->
   <xacro:kinect name="openni" parent="tower_link">
-    <origin xyz="-0.001 -0.03 0.49" rpy="0.0 0.545 0.0" />
+    <origin xyz="0.0509 -0.03 0.49" rpy="0.0 0.545 0.0" />
   </xacro:kinect>
   -->
