Commit message: update asus xtion model

File: raw_common/raw_robot_description/urdf/sensors/asus_xtion.gazebo.xacro (robot description, xacro)
@@ -4,5 +4,5 @@
       xmlns:interface="http://playerstage.sourceforge.net/gazebo/xmlschema/#interface"
       xmlns:xacro="http://ros.org/wiki/xacro">
-<xacro:macro name="asus_xtion_gazebo" params="name ros_topic">
+<xacro:macro name="asus_xtion_gazebo" params="name">
   <gazebo reference="openni_camera">
     <sensor:ray name="${name}_sensor">
@@ -26,5 +26,5 @@
             <alwaysOn>true</alwaysOn>
             <updateRate>10</updateRate> <!-- true value 30Hz -->
-            <topicName>${ros_topic}</topicName>
+            <topicName>/camera/depth/points</topicName>
             <frameName>openni_camera</frameName>
             <interface:laser name="${name}_ray_block_iface" />

File: raw_common/raw_robot_description/urdf/sensors/asus_xtion.urdf.xacro (robot description, xacro)
@@ -33,5 +33,5 @@
 		</joint>
 	</xacro:macro>
-  <xacro:macro name="asus_xtion" params="name parent *origin ros_topic tilt">
+  <xacro:macro name="asus_xtion" params="name parent *origin tilt">
   	<link name="${name}_foot_link">
       <inertial>
@@ -41,14 +41,14 @@
       </inertial>
       <visual>
-        <origin xyz="0 0 0" rpy="0 0 0" />
+        <origin xyz="0 0 0" rpy="${M_PI/2} 0 ${M_PI/2}" />
         <geometry>
-          <box size="0.05 0.088 0.005"/>
+           <mesh filename="package://raw_robot_description/meshes/sensors/asus_xtion_pro_live_base.dae" scale="0.0005 0.0008 0.001"/>
         </geometry>
-        <material name="Red" />
+        <material name="Black" />
       </visual>
       <collision>
-        <origin xyz="0 0 0" rpy="0 0 0" />
+        <origin xyz="0 0 0" rpy="${M_PI/2} 0 ${M_PI/2}" />
         <geometry>
-           <box size="0.05 0.088 0.005"/>
+           <mesh filename="package://raw_robot_description/meshes/sensors/asus_xtion_pro_live_base.dae" scale="0.0005 0.001 0.001"/>
         </geometry>
       </collision >
@@ -59,5 +59,5 @@
       <child link="${name}_foot_link"/>
     </joint>
-    <link name="asus_xtion_tilt_link">
+    <link name="${name}_tilt_link">
       <inertial>
         <mass value="0.01" />
@@ -82,5 +82,5 @@
     <joint name="asus_xtion_tilt_joint" type="fixed">
      	<parent link="${name}_foot_link"/>
-     	<child link="asus_xtion_tilt_link"/>
+     	<child link="${name}_tilt_link"/>
      	<!--<axis xyz="0 1 0"/>-->
       	<origin xyz="0 0 0.0075" rpy="0 ${tilt} 0"/>
@@ -94,14 +94,14 @@
       </inertial>
       <visual>
-        <origin xyz="0 -0.03 0" rpy="0 0 0" />
+        <origin xyz="0.01 -0.03 0" rpy="${M_PI/2} 0 ${M_PI/2}" />
         <geometry>
-          <box size="0.05 0.18 0.035"/>
+          <mesh filename="package://raw_robot_description/meshes/sensors/asus_xtion_pro_live_camera.dae" scale="0.001 0.001 0.001"/>
         </geometry>
-        <material name="Red" />
+        <material name="Black" />
       </visual>
       <collision>
-        <origin xyz="0 -0.03 0" rpy="0 0 0" />
+        <origin xyz="0.01 -0.03 0" rpy="${M_PI/2} 0 ${M_PI/2}" />
         <geometry>
-           <box size="0.05 0.18 0.035"/>
+           <mesh filename="package://raw_robot_description/meshes/sensors/asus_xtion_pro_live_camera.dae" scale="0.001 0.001 0.001"/>
         </geometry>
       </collision >
@@ -109,5 +109,5 @@
     <joint name="${name}_camera_joint" type="fixed">
       <origin xyz="0 0.03 0.03" rpy="0 0 0" />
-      <parent link="asus_xtion_tilt_link"/>
+      <parent link="${name}_tilt_link"/>
       <child link="${name}_camera"/>
     </joint>
@@ -122,5 +122,5 @@
 	</xacro:asus_xtion_eye>
    <!-- for simulation -->
-   <xacro:asus_xtion_gazebo name="${name}" ros_topic="${ros_topic}"/>
+   <xacro:asus_xtion_gazebo name="${name}"/>
   </xacro:macro>
 </root>
