Commit message: move kinect meshes to sensors

File: raw_common/raw_robot_description/urdf/sensors/kinect.urdf.xacro (robot description, xacro)
@@ -18,7 +18,7 @@
     </inertial>
     <visual>
-      <origin xyz=" 0 0 0 " rpy="0 0 0" />
+      <origin xyz="0.0 0.0 0.0" rpy="0 0 0" />
       <geometry>
-       <mesh filename="package://raw_robot_description/meshes/kinect/kinect.dae"/>
+       <mesh filename="package://raw_robot_description/meshes/sensors/kinect.dae"/>
       </geometry>
     </visual>
@@ -26,5 +26,5 @@
       <origin xyz="0.0 0.0 0.0" rpy="0 0 0" />
       <geometry>
-        <box size="0.0730 .2760 0.0720"/>
+        <mesh filename="package://raw_robot_description/meshes/sensors/kinect.dae"/>
       </geometry>
     </collision>
