Commit message: change package name from raw_description to raw_robot_description because of conflicts with the same package in cob_common

File: raw_common/raw_robot_description/urdf/sensors/asus_xtion.urdf.xacro (robot description, xacro)
@@ -1,5 +1,5 @@
 <?xml version="1.0"?>
 <root xmlns:xacro="http://playerstage.sourceforge.net/gazebo/xmlschema/#interface">
-  <include filename="$(find raw_description)/urdf/sensors/asus_xtion.gazebo.xacro" />
+  <include filename="$(find raw_robot_description)/urdf/sensors/asus_xtion.gazebo.xacro" />
   <property name="eye_radius" value="0.0095" />
   <property name="eye_length" value="0.002" />

File: raw_common/raw_robot_description/urdf/sensors/kinect.urdf.xacro (robot description, xacro)
@@ -2,5 +2,5 @@
 <robot name="kinect_hardware" xmlns:xacro="http://ros.org/wiki/xacro">
   <property name="M_PI" value="3.14159"/>
-  <include filename="$(find raw_description)/urdf/sensors/kinect.gazebo.xacro"/>
+  <include filename="$(find raw_robot_description)/urdf/sensors/kinect.gazebo.xacro"/>
   <xacro:macro name="kinect" params="name parent *origin">
    <joint name="${name}_camera_joint" type="fixed">
@@ -20,5 +20,5 @@
       <origin xyz=" 0 0 0 " rpy="0 0 0" />
       <geometry>
-       <mesh filename="package://raw_description/meshes/kinect/kinect.dae"/>
+       <mesh filename="package://raw_robot_description/meshes/kinect/kinect.dae"/>
       </geometry>
     </visual>

File: raw_common/raw_robot_description/urdf/tower/cam3d_tower.urdf.xacro (robot description, xacro)
@@ -4,5 +4,5 @@
        xmlns:interface="http://playerstage.sourceforge.net/gazebo/xmlschema/#interface"
        xmlns:xacro="http://ros.org/wiki/xacro">
-  <include filename="$(find raw_description)/urdf/sensors/kinect.urdf.xacro" />
+  <include filename="$(find raw_robot_description)/urdf/sensors/kinect.urdf.xacro" />
   <property name="height" value="0.515" />
   <property name="width" value="0.03" />

File: raw_robots/raw_hardware_config/youbot-hbrs2/urdf/youbot-hbrs2.urdf.xacro (robot description, xacro)
@@ -40,6 +40,6 @@
   </xacro:youbot_gripper>
   <!-- BRSU SPECIFIC STUFF -->
-  <include filename="$(find raw_description)/urdf/materials.urdf.xacro" />
-  <include filename="$(find raw_description)/urdf/tower/cam3d_tower.urdf.xacro" />
+  <include filename="$(find raw_robot_description)/urdf/materials.urdf.xacro" />
+  <include filename="$(find raw_robot_description)/urdf/tower/cam3d_tower.urdf.xacro" />
   <!--include filename="$(find youbot_description)/urdf/sensors/asus_xtion.urdf.xacro" />-->
   <!-- base laser rear -->

Commit message: adapt asus model and position

File: raw_common/raw_robot_description/urdf/sensors/asus_xtion.urdf.xacro (robot description, xacro)
@@ -2,6 +2,4 @@
 <root xmlns:xacro="http://playerstage.sourceforge.net/gazebo/xmlschema/#interface">
   <include filename="$(find raw_robot_description)/urdf/sensors/asus_xtion.gazebo.xacro" />
-  <property name="eye_radius" value="0.0095" />
-  <property name="eye_length" value="0.002" />
   <property name="eye_x_offset" value="0.025" />
   <property name="eye_y_offset" value="0.035" />
@@ -9,21 +7,8 @@
 		<link name="${parent}_${suffix}_link">
 			<inertial>
-				<mass value="1" />
+				<mass value="0.01" />
 				<origin xyz="0 0 0" />
 				<inertia ixx="0.1" ixy="0" ixz="0" iyy="0.1" iyz="0" izz="0.1" />
 			</inertial>
-			<visual>
-				<origin xyz="0 0 0" rpy="0 0 0" />
-		        <geometry>
-		          	<cylinder length="${eye_length}" radius="${eye_radius}"/>
-		        </geometry>
-		        <material name="Blue" />
-			</visual>
-			<collision>
-				<origin xyz="0 0 0" rpy="0 0 0" />
-		        <geometry>
-		          	<cylinder length="${eye_length}" radius="${eye_radius}"/>
-		        </geometry>
-			</collision>
 		</link>
 		<joint name="${parent}_${suffix}_joint" type="fixed">
@@ -36,19 +21,19 @@
   	<link name="${name}_foot_link">
       <inertial>
-        <mass value="0.01" />
+        <mass value="0.05" />
         <origin xyz="0 0 0" rpy="0 0 0"/>
         <inertia ixx="0.0001" ixy="0" ixz="0" iyy="0.0001" iyz="0" izz="0.0001" />
       </inertial>
       <visual>
-        <origin xyz="0 0 0" rpy="${M_PI/2} 0 ${M_PI/2}" />
+        <origin xyz="0.01 0 0" rpy="${M_PI/2} 0 ${M_PI/2}" />
         <geometry>
-           <mesh filename="package://raw_robot_description/meshes/sensors/asus_xtion_pro_live_base.dae" scale="0.0005 0.0008 0.001"/>
+           <mesh filename="package://raw_robot_description/meshes/sensors/asus_xtion_pro_live_base.dae" scale="0.0004 0.0007 0.001"/>
         </geometry>
         <material name="Black" />
       </visual>
       <collision>
-        <origin xyz="0 0 0" rpy="${M_PI/2} 0 ${M_PI/2}" />
+        <origin xyz="0.01 0 0" rpy="${M_PI/2} 0 ${M_PI/2}" />
         <geometry>
-           <mesh filename="package://raw_robot_description/meshes/sensors/asus_xtion_pro_live_base.dae" scale="0.0005 0.001 0.001"/>
+           <mesh filename="package://raw_robot_description/meshes/sensors/asus_xtion_pro_live_base.dae" scale="0.0004 0.0007 0.001"/>
         </geometry>
       </collision >
@@ -89,10 +74,10 @@
     <link name="${name}_camera">
       <inertial>
-        <mass value="0.01" />
+        <mass value="0.1" />
         <origin xyz="0 0 0" rpy="0 0 0"/>
         <inertia ixx="0.0001" ixy="0" ixz="0" iyy="0.0001" iyz="0" izz="0.0001" />
       </inertial>
       <visual>
-        <origin xyz="0.01 -0.03 0" rpy="${M_PI/2} 0 ${M_PI/2}" />
+        <origin xyz="0.02 -0.03 0" rpy="${M_PI/2} 0 ${M_PI/2}" />
         <geometry>
           <mesh filename="package://raw_robot_description/meshes/sensors/asus_xtion_pro_live_camera.dae" scale="0.001 0.001 0.001"/>
@@ -101,5 +86,5 @@
       </visual>
       <collision>
-        <origin xyz="0.01 -0.03 0" rpy="${M_PI/2} 0 ${M_PI/2}" />
+        <origin xyz="0.02 -0.03 0" rpy="${M_PI/2} 0 ${M_PI/2}" />
         <geometry>
            <mesh filename="package://raw_robot_description/meshes/sensors/asus_xtion_pro_live_camera.dae" scale="0.001 0.001 0.001"/>

File: raw_robots/raw_hardware_config/youbot-hbrs2/urdf/youbot-hbrs2.urdf.xacro (robot description, xacro)
@@ -49,5 +49,5 @@
      <origin xyz="-0.3 0.0 -0.03" rpy="0 0 ${M_PI}" />
   </xacro:hokuyo_urg04_laser>
-  <!-- Sensor angle on arm-->
+  <!-- Sensor angle on arm -->
   <xacro:sensor_angle name="arm_sensor_angle" parent="arm_link_5">
     <origin xyz="-0.002 0.0 -0.023" rpy="0.0 0.0 0.0" />
@@ -55,5 +55,5 @@
   <!-- ASUS Xtion on arm sensor angle -->
   <xacro:asus_xtion name="openni" parent="arm_sensor_angle_part2_link" tilt="0.0">
-    <origin xyz="0.0 0.0 0.0" rpy="${M_PI} 0.0 ${M_PI}" />
+    <origin xyz="0.01 0.0 0.0" rpy="${M_PI} 0.0 ${M_PI}" />
   </xacro:asus_xtion>
   <!-- tower with 3D camera
