Commit message: update kinect model

File: raw_common/raw_robot_description/urdf/sensors/kinect_camera.urdf.xacro (robot description, xacro)
@@ -1,7 +1,9 @@
 <?xml version="1.0"?>
-<robot name="kinect_hardware" xmlns:xacro="http://ros.org/wiki/xacro">
-  <property name="M_PI" value="3.14159"/>
-  <include filename="$(find raw_robot_description)/urdf/sensors/kinect.gazebo.xacro"/>
-  <xacro:macro name="kinect" params="name parent *origin">
+<root xmlns:sensor="http://playerstage.sourceforge.net/gazebo/xmlschema/#sensor"
+      xmlns:controller="http://playerstage.sourceforge.net/gazebo/xmlschema/#controller"
+      xmlns:interface="http://playerstage.sourceforge.net/gazebo/xmlschema/#interface"
+      xmlns:xacro="http://ros.org/wiki/xacro">
+  <include filename="$(find raw_robot_description)/urdf/sensors/kinect_camera.gazebo.xacro"/>
+  <xacro:macro name="kinect_camera" params="name parent *origin">
    <joint name="${name}_camera_joint" type="fixed">
     <insert_block name="origin" />
@@ -87,5 +89,5 @@
   </link>
   <!-- for simulation -->
-  <xacro:kinect_gazebo frame_rate="10.0" />
+  <xacro:kinect_camera_gazebo name="openni" />
 </xacro:macro>
-</robot>
+</root>
