Commit message: rename properties, since they have the same name and will be overwritten by the other ones

File: raw_common/raw_robot_description/urdf/misc/cam3d_tower.urdf.xacro (robot description, xacro)
@@ -4,25 +4,25 @@
        xmlns:interface="http://playerstage.sourceforge.net/gazebo/xmlschema/#interface"
        xmlns:xacro="http://ros.org/wiki/xacro">
-  <property name="height" value="0.49" />
-  <property name="width" value="0.03" />
-  <property name="depth" value="0.03" />
+  <property name="cam3d_tower_height" value="0.49" />
+  <property name="cam3d_tower_width" value="0.03" />
+  <property name="cam3d_tower_depth" value="0.03" />
   <xacro:macro name="cam3d_tower" params="name parent *origin">
   	<link name="${name}_link">
       <inertial>
         <mass value="0.01" />
-        <origin xyz="0 0 ${(height/2) - height}" rpy="0 0 0"/>
+        <origin xyz="0 0 ${(cam3d_tower_height/2) - cam3d_tower_height}" rpy="0 0 0"/>
         <inertia ixx="0.0001" ixy="0" ixz="0" iyy="0.0001" iyz="0" izz="0.0001" />
       </inertial>
       <visual>
-        <origin xyz="0 0 ${height - (height/2)}" rpy="0 0 0" />
+        <origin xyz="0 0 ${cam3d_tower_height - (cam3d_tower_height/2)}" rpy="0 0 0" />
         <geometry>
-          <box size="${depth} ${width} ${height}"/>
+          <box size="${cam3d_tower_depth} ${cam3d_tower_width} ${cam3d_tower_height}"/>
         </geometry>
         <material name="LightGrey" />
       </visual>
       <collision>
-        <origin xyz="0 0 ${height - (height/2)}" rpy="0 0 0" />
+        <origin xyz="0 0 ${cam3d_tower_height - (cam3d_tower_height/2)}" rpy="0 0 0" />
         <geometry>
-           <box size="${depth} ${width} ${height}"/>
+           <box size="${cam3d_tower_depth} ${cam3d_tower_width} ${cam3d_tower_height}"/>
         </geometry>
       </collision >

File: raw_common/raw_robot_description/urdf/misc/sensor_angle.urdf.xacro (robot description, xacro)
@@ -4,7 +4,7 @@
        xmlns:interface="http://playerstage.sourceforge.net/gazebo/xmlschema/#interface"
        xmlns:xacro="http://ros.org/wiki/xacro">
-	<property name="width"  value="0.097" />
-	<property name="height" value="0.0015" />
-	<property name="depth"  value="0.0625" />
+	<property name="sensor_angle_width"  value="0.097" />
+	<property name="sensor_angle_height" value="0.0015" />
+	<property name="sensor_angle_depth"  value="0.0625" />
 	<xacro:macro name="sensor_angle" params="name parent *origin">
 		<link name="${name}_part1_link">
@@ -17,5 +17,5 @@
 				<origin xyz="0 0 0" rpy="0 0 0" />
 				<geometry>
-					<box size="${depth} ${width} ${height}"/>
+					<box size="${sensor_angle_depth} ${sensor_angle_width} ${sensor_angle_height}"/>
 				</geometry>
 				<material name="Black" />
@@ -24,5 +24,5 @@
 				<origin xyz="0 0 0" rpy="0 0 0" />
 				<geometry>
-					<box size="${depth} ${width} ${height}"/>
+					<box size="${sensor_angle_depth} ${sensor_angle_width} ${sensor_angle_height}"/>
 				</geometry>
 			</collision >
@@ -42,5 +42,5 @@
 				<origin xyz="0 0 0" rpy="0 0 0" />
 				<geometry>
-					<box size="${depth} ${width} ${height}"/>
+					<box size="${sensor_angle_depth} ${sensor_angle_width} ${sensor_angle_height}"/>
 				</geometry>
 				<material name="Black" />
@@ -49,10 +49,10 @@
 				<origin xyz="0 0 0" rpy="0 0 0" />
 				<geometry>
-					<box size="${depth} ${width} ${height}"/>
+					<box size="${sensor_angle_depth} ${sensor_angle_width} ${sensor_angle_height}"/>
 				</geometry>
 			</collision >
 		</link>
 		<joint name="${name}_part2_joint" type="fixed">
-			<origin xyz="${-((depth/2) - (height/2))} 0 ${((depth/2) - (height/2))}" rpy="0 ${M_PI/2} 0 "/>
+			<origin xyz="${-((sensor_angle_depth/2) - (sensor_angle_height/2))} 0 ${((sensor_angle_depth/2) - (sensor_angle_height/2))}" rpy="0 ${M_PI/2} 0 "/>
 			<parent link="${name}_part1_link"/>
 			<child link="${name}_part2_link"/>
