Commit message: adjust kinect pose

File: raw_robots/raw_hardware_config/youbot-hbrs2/urdf/youbot-hbrs2.urdf.xacro (robot description, xacro)
@@ -52,6 +52,6 @@
   </xacro:cam3d_tower>
   <!-- 3D camera on tower -->
-  <xacro:kinect name="openni" parent="plate_link">
-    <origin xyz="-0.010 0.008 0.422" rpy="-0.048 0.419 0.031" />
+  <xacro:kinect name="openni" parent="tower_link">
+    <origin xyz="0.05 0.0 0.515" rpy="0.0 0.61 0.0" />
   </xacro:kinect>
   -->

Commit message: calibrated kinect position

File: raw_robots/raw_hardware_config/youbot-hbrs2/urdf/youbot-hbrs2.urdf.xacro (robot description, xacro)
@@ -53,5 +53,5 @@
   <!-- 3D camera on tower -->
   <xacro:kinect name="openni" parent="tower_link">
-    <origin xyz="0.05 0.0 0.515" rpy="0.0 0.61 0.0" />
+    <origin xyz="0.0 -0.03 0.505" rpy="0.0 0.55 0.0" />
   </xacro:kinect>
   -->

Commit message: new calibrated pose for kinect on tower

File: raw_robots/raw_hardware_config/youbot-hbrs2/urdf/youbot-hbrs2.urdf.xacro (robot description, xacro)
@@ -53,5 +53,5 @@
   <!-- 3D camera on tower -->
   <xacro:kinect name="openni" parent="tower_link">
-    <origin xyz="0.0 -0.03 0.505" rpy="0.0 0.55 0.0" />
+    <origin xyz="-0.001 -0.03 0.49" rpy="0.0 0.545 0.0" />
   </xacro:kinect>
   -->

Commit message: remove cam3d tower and add sensor angle and asus to the arm

File: raw_robots/raw_hardware_config/youbot-hbrs2/urdf/youbot-hbrs2.urdf.xacro (robot description, xacro)
@@ -41,17 +41,29 @@
   <!-- BRSU SPECIFIC STUFF -->
   <include filename="$(find raw_robot_description)/urdf/materials.urdf.xacro" />
-  <include filename="$(find raw_robot_description)/urdf/misc/cam3d_tower.urdf.xacro" />
-  <include filename="$(find raw_robot_description)/urdf/sensors/kinect.urdf.xacro" />
+  <include filename="$(find raw_robot_description)/urdf/misc/sensor_angle.urdf.xacro" />
+  <include filename="$(find raw_robot_description)/urdf/sensors/asus_xtion.urdf.xacro" />
+  <!-- include filename="$(find raw_robot_description)/urdf/misc/cam3d_tower.urdf.xacro" />
+  <include filename="$(find raw_robot_description)/urdf/sensors/kinect.urdf.xacro" /-->
   <!-- base laser rear -->
   <xacro:hokuyo_urg04_laser name="base_laser_rear" parent="base" ros_topic="scan_rear" update_rate="10" min_angle="-1.57" max_angle="1.57" >
-     <origin xyz="-0.3 0 -0.03" rpy="0 0 ${M_PI}" />
+     <origin xyz="-0.3 0.0 -0.03" rpy="0 0 ${M_PI}" />
   </xacro:hokuyo_urg04_laser>
-  <!-- tower with 3D camera -->
+  <!-- Sensor angle on arm-->
+  <xacro:sensor_angle name="arm_sensor_angle" parent="arm_link_5">
+    <origin xyz="-0.002 0.0 -0.023" rpy="0.0 0.0 0.0" />
+  </xacro:sensor_angle>
+  <!-- ASUS Xtion on arm sensor angle -->
+  <xacro:asus_xtion name="openni" parent="arm_sensor_angle_part2_link" tilt="0.0">
+    <origin xyz="0.0 0.0 0.0" rpy="${M_PI} 0.0 ${M_PI}" />
+  </xacro:asus_xtion>
+  <!-- tower with 3D camera
   <xacro:cam3d_tower name="tower" parent="plate_link">
     <origin xyz="-0.0659 0.0 0.025" rpy="0 0 0" />
   </xacro:cam3d_tower>
-  <!-- 3D camera on tower -->
+  -->
+  <!-- 3D camera on tower
   <xacro:kinect name="openni" parent="tower_link">
     <origin xyz="0.0509 -0.03 0.49" rpy="0.0 0.545 0.0" />
   </xacro:kinect>
+  -->
 </robot>

Commit message: change names

File: raw_robots/raw_hardware_config/youbot-hbrs2/urdf/youbot-hbrs2.urdf.xacro (robot description, xacro)
@@ -42,7 +42,7 @@
   <include filename="$(find raw_robot_description)/urdf/materials.urdf.xacro" />
   <include filename="$(find raw_robot_description)/urdf/misc/sensor_angle.urdf.xacro" />
-  <include filename="$(find raw_robot_description)/urdf/sensors/asus_xtion.urdf.xacro" />
-  <!-- include filename="$(find raw_robot_description)/urdf/misc/cam3d_tower.urdf.xacro" />
-  <include filename="$(find raw_robot_description)/urdf/sensors/kinect.urdf.xacro" /-->
+  <include filename="$(find raw_robot_description)/urdf/sensors/asus_xtion_camera.urdf.xacro" />
+  <!-- include filename="$(find raw_robot_description)/urdf/misc/cam3d_tower.urdf.xacro" /-->
+  <!-- include filename="$(find raw_robot_description)/urdf/sensors/kinect_camera.urdf.xacro" /-->
   <!-- base laser rear -->
   <xacro:hokuyo_urg04_laser name="base_laser_rear" parent="base" ros_topic="scan_rear" update_rate="10" min_angle="-1.57" max_angle="1.57" >
@@ -54,7 +54,7 @@
   </xacro:sensor_angle>
   <!-- ASUS Xtion on arm sensor angle -->
-  <xacro:asus_xtion name="openni" parent="arm_sensor_angle_part2_link" tilt="0.0">
+  <xacro:asus_xtion_camera name="openni" parent="arm_sensor_angle_part2_link"  tilt="0.0">
     <origin xyz="0.01 0.0 0.0" rpy="${M_PI} 0.0 ${M_PI}" />
-  </xacro:asus_xtion>
+  </xacro:asus_xtion_camera>
   <!-- tower with 3D camera
   <xacro:cam3d_tower name="tower" parent="plate_link">
@@ -63,7 +63,6 @@
   -->
   <!-- 3D camera on tower
-  <xacro:kinect name="openni" parent="tower_link">
-    <origin xyz="0.0509 -0.03 0.49" rpy="0.0 0.545 0.0" />
-  </xacro:kinect>
-  -->
+  <xacro:kinect_camera name="openni" parent="arm_sensor_angle_part2_link">
+    <origin xyz="0.01 0.0 0.0" rpy="${M_PI} 0.0 ${M_PI}" />
+  </xacro:kinect_camera> -->
 </robot>

Commit message: add kinect tower and remove asus from arm

File: raw_robots/raw_hardware_config/youbot-hbrs2/urdf/youbot-hbrs2.urdf.xacro (robot description, xacro)
@@ -42,7 +42,7 @@
   <include filename="$(find raw_robot_description)/urdf/materials.urdf.xacro" />
   <include filename="$(find raw_robot_description)/urdf/misc/sensor_angle.urdf.xacro" />
-  <include filename="$(find raw_robot_description)/urdf/sensors/asus_xtion_camera.urdf.xacro" />
-  <!-- include filename="$(find raw_robot_description)/urdf/misc/cam3d_tower.urdf.xacro" /-->
-  <!-- include filename="$(find raw_robot_description)/urdf/sensors/kinect_camera.urdf.xacro" /-->
+  <include filename="$(find raw_robot_description)/urdf/misc/cam3d_tower.urdf.xacro" />
+  <include filename="$(find raw_robot_description)/urdf/sensors/kinect_camera.urdf.xacro" />
+  <!--include filename="$(find raw_robot_description)/urdf/sensors/asus_xtion_camera.urdf.xacro" /-->
   <!-- base laser rear -->
   <xacro:hokuyo_urg04_laser name="base_laser_rear" parent="base" ros_topic="scan_rear" update_rate="10" min_angle="-1.57" max_angle="1.57" >
@@ -54,15 +54,14 @@
   </xacro:sensor_angle>
   <!-- ASUS Xtion on arm sensor angle -->
-  <xacro:asus_xtion_camera name="openni" parent="arm_sensor_angle_part2_link"  tilt="0.0">
+  <!--xacro:asus_xtion_camera name="openni" parent="arm_sensor_angle_part2_link"  tilt="0.0">
     <origin xyz="0.01 0.0 0.0" rpy="${M_PI} 0.0 ${M_PI}" />
-  </xacro:asus_xtion_camera>
-  <!-- tower with 3D camera
+  </xacro:asus_xtion_camera-->
+  <!-- tower -->
   <xacro:cam3d_tower name="tower" parent="plate_link">
     <origin xyz="-0.0659 0.0 0.025" rpy="0 0 0" />
   </xacro:cam3d_tower>
-  -->
-  <!-- 3D camera on tower
-  <xacro:kinect_camera name="openni" parent="arm_sensor_angle_part2_link">
-    <origin xyz="0.01 0.0 0.0" rpy="${M_PI} 0.0 ${M_PI}" />
-  </xacro:kinect_camera> -->
+  <!-- 3D camera on tower -->
+  <xacro:kinect_camera name="openni" parent="tower_link">
+    <origin xyz="0.0509 -0.03 0.49" rpy="0 0.545 0" />
+  </xacro:kinect_camera>
 </robot>

Commit message: add model of microsoft lifecam to the youbot-hbrs2

File: raw_robots/raw_hardware_config/youbot-hbrs2/urdf/youbot-hbrs2.urdf.xacro (robot description, xacro)
@@ -44,4 +44,5 @@
   <include filename="$(find raw_robot_description)/urdf/misc/cam3d_tower.urdf.xacro" />
   <include filename="$(find raw_robot_description)/urdf/sensors/kinect_camera.urdf.xacro" />
+  <include filename="$(find raw_robot_description)/urdf/sensors/microsoft_lifecam.urdf.xacro" />
   <!--include filename="$(find raw_robot_description)/urdf/sensors/asus_xtion_camera.urdf.xacro" /-->
   <!-- base laser rear -->
@@ -65,3 +66,7 @@
     <origin xyz="0.0509 -0.03 0.49" rpy="0 0.545 0" />
   </xacro:kinect_camera>
+  <!-- Microsoft LifeCam on gripper -->
+  <xacro:microsoft_lifecam name="microsoft_lifecam" parent="arm_sensor_angle_part2_link">
+    <origin xyz="-0.04 0 -0.03" rpy="0 ${M_PI} 0" />
+  </xacro:microsoft_lifecam>
 </robot>
