Commit message: update collision model of the objects

File: raw_simulation/raw_gazebo_objects/ros/objects/adapter_sleeve_r20.urdf.xacro (robot description, xacro)
@@ -2,4 +2,4 @@
 <robot name="adapter_sleeve_r20" xmlns:xacro="http://ros.org/wiki/xacro">
 	<include filename="$(find raw_gazebo_objects)/ros/templates/model.urdf.xacro" />
-	<xacro:model_template name="adapter_sleeve_r20" model_filename="adapter_sleeve_r20.dae" scale="0.001" height="0.045" weight="0.010"/>
+	<xacro:model_template name="adapter_sleeve_r20" model_filename="adapter_sleeve_r20.dae" scale="0.001" height="0.045" width="0.03" depth="0.03" weight="0.010"/>
 </robot>

File: raw_simulation/raw_gazebo_objects/ros/objects/adapter_sleeve_v20.urdf.xacro (robot description, xacro)
@@ -2,4 +2,4 @@
 <robot name="adapter_sleeve_v20" xmlns:xacro="http://ros.org/wiki/xacro">
 	<include filename="$(find raw_gazebo_objects)/ros/templates/model.urdf.xacro" />
-	<xacro:model_template name="adapter_sleeve_v20" model_filename="adapter_sleeve_v20.dae" scale="0.001" height="0.045"  weight="0.015"/>
+	<xacro:model_template name="adapter_sleeve_v20" model_filename="adapter_sleeve_v20.dae" scale="0.001" height="0.045" width="0.03" depth="0.03" weight="0.015"/>
 </robot>

File: raw_simulation/raw_gazebo_objects/ros/objects/aluprofil_f20_100_gray.urdf.xacro (robot description, xacro)
@@ -2,4 +2,4 @@
 <robot name="aluprofil_f20_100_gray" xmlns:xacro="http://ros.org/wiki/xacro">
 	<include filename="$(find raw_gazebo_objects)/ros/templates/model.urdf.xacro" />
-	<xacro:model_template name="aluprofil_f20_100_gray" model_filename="aluprofil_f20_100_gray.dae" scale="0.001"  height="0.1"  weight="0.05"/>
+	<xacro:model_template name="aluprofil_f20_100_gray" model_filename="aluprofil_f20_100_gray.dae" scale="0.001"  height="0.1" width="0.02" depth="0.02" weight="0.05"/>
 </robot>

File: raw_simulation/raw_gazebo_objects/ros/objects/aluprofil_s40_100_gray.urdf.xacro (robot description, xacro)
@@ -2,4 +2,4 @@
 <robot name="aluprofil_s40_100_gray" xmlns:xacro="http://ros.org/wiki/xacro">
 	<include filename="$(find raw_gazebo_objects)/ros/templates/model.urdf.xacro" />
-	<xacro:model_template name="aluprofil_s40_100_gray" model_filename="aluprofil_s40_100_gray.dae" scale="0.001"  height="0.1"  weight="0.185"/>
+	<xacro:model_template name="aluprofil_s40_100_gray" model_filename="aluprofil_s40_100_gray.dae" scale="0.001"  height="0.1" width="0.04" depth="0.04" weight="0.185"/>
 </robot>

File: raw_simulation/raw_gazebo_objects/ros/objects/bolt_m20_100.urdf.xacro (robot description, xacro)
@@ -2,4 +2,4 @@
 <robot name="bolt_m20_100" xmlns:xacro="http://ros.org/wiki/xacro">
 	<include filename="$(find raw_gazebo_objects)/ros/templates/model.urdf.xacro" />
-	<xacro:model_template name="bolt_m20_100" model_filename="bolt_m20_100.dae" scale="0.001"  height="0.01"  weight="0.290"/>
+	<xacro:model_template name="bolt_m20_100" model_filename="bolt_m20_100.dae" scale="0.001"  height="0.11" width="0.02" depth="0.02" weight="0.290"/>
 </robot>

File: raw_simulation/raw_gazebo_objects/ros/objects/bolt_m20_180.urdf.xacro (robot description, xacro)
@@ -2,4 +2,4 @@
 <robot name="bolt_m20_180" xmlns:xacro="http://ros.org/wiki/xacro">
 	<include filename="$(find raw_gazebo_objects)/ros/templates/model.urdf.xacro" />
-	<xacro:model_template name="bolt_m20_180" model_filename="bolt_m20_180.dae" scale="0.001"  height="0.01"  weight="0.477"/>
+	<xacro:model_template name="bolt_m20_180" model_filename="bolt_m20_180.dae" scale="0.001"  height="0.11" width="0.02" depth="0.02" weight="0.477"/>
 </robot>

File: raw_simulation/raw_gazebo_objects/ros/objects/nut_m20.urdf.xacro (robot description, xacro)
@@ -2,4 +2,4 @@
 <robot name="nut_m20" xmlns:xacro="http://ros.org/wiki/xacro">
 	<include filename="$(find raw_gazebo_objects)/ros/templates/model.urdf.xacro" />
-	<xacro:model_template name="nut_m20" model_filename="nut_m20.dae" scale="0.001"  height="0.01"  weight="0.068"/>
+	<xacro:model_template name="nut_m20" model_filename="nut_m20.dae" scale="0.001"  height="0.015" width="0.028" depth="0.028" weight="0.068"/>
 </robot>

File: raw_simulation/raw_gazebo_objects/ros/objects/nut_m30.urdf.xacro (robot description, xacro)
@@ -2,4 +2,4 @@
 <robot name="nut_m30" xmlns:xacro="http://ros.org/wiki/xacro">
 	<include filename="$(find raw_gazebo_objects)/ros/templates/model.urdf.xacro" />
-	<xacro:model_template name="nut_m30" model_filename="nut_m30.dae" scale="0.001"  height="0.01"  weight="0.215"/>
+	<xacro:model_template name="nut_m30" model_filename="nut_m30.dae" scale="0.001"  height="0.025" width="0.045" depth="0.045"  weight="0.215"/>
 </robot>

File: raw_simulation/raw_gazebo_objects/ros/templates/model.urdf.xacro (robot description, xacro)
@@ -14,5 +14,5 @@
 	    xmlns:physics="http://playerstage.sourceforge.net/gazebo/xmlschema/#physics"
 	    xmlns:xacro="http://www.ros.org/wiki/xacro">
-	<xacro:macro name="model_template" params="name model_filename scale height weight">
+	<xacro:macro name="model_template" params="name model_filename scale height width depth weight">
 		<link name="${name}_link">
 			<inertial>
@@ -30,5 +30,5 @@
 				<origin xyz="0 0 ${-height / 2}" rpy="0 0 0" />
 				<geometry>
-					<mesh filename="package://raw_gazebo_objects/common/models/${model_filename}" scale="${scale} ${scale} ${scale}" />
+					<box size="${height} ${width} ${depth}"/>
 				</geometry>
 			</collision >
